File: UART Card.kicad_pcb (KiCad board)
At the start: 2 copper layers, 100 x 100 mm, 30 parts, among them J1 Conn_02x20_Odd_Even, J2 DB9_ Male, U1 74LS00, U2 MAX232, U3 CDP1854AE, U4 74LS393, U5 74LS157, U6 MCP2221AxP, X1 CXO_DIP8

Commit message: Disconnect ~CLEAR from USB Controller
Parts:
- added R3: 10K, Resistor_THT:R_Axial_DIN0207_L6.3mm_D2.5mm_P7.62mm_Horizontal, F.Cu at (143.9, 105.2)
Connections:
- net ~EF4 renamed ~{EF4}
- net ~INTERRUPT renamed ~{INTERRUPT}
- net ~MRD renamed ~{MRD}
- net ~N3 renamed ~{N3}
- J1 pad 11: SC0 -> unconnected-(J1-Pin_11-Pad11)
- J1 pad 12: ~MWR -> unconnected-(J1-Pin_12-Pad12)
- J1 pad 14: TPA -> unconnected-(J1-Pin_14-Pad14)
- J1 pad 25: ~IOW -> unconnected-(J1-Pin_25-Pad25)
- J1 pad 26: ~IOR -> unconnected-(J1-Pin_26-Pad26)
- J1 pad 27: ~N7 -> unconnected-(J1-Pin_27-Pad27)
- J1 pad 28: ~N6 -> unconnected-(J1-Pin_28-Pad28)
- J1 pad 29: ~N5 -> unconnected-(J1-Pin_29-Pad29)
- J1 pad 3: ~WAIT -> unconnected-(J1-Pin_3-Pad3)
- J1 pad 30: ~N4 -> unconnected-(J1-Pin_30-Pad30)
- J1 pad 32: ~N2 -> unconnected-(J1-Pin_32-Pad32)
- J1 pad 33: ~N1 -> unconnected-(J1-Pin_33-Pad33)
- J1 pad 35: ~EF1 -> unconnected-(J1-Pin_35-Pad35)
- J1 pad 36: ~EF2 -> unconnected-(J1-Pin_36-Pad36)
- J1 pad 37: ~EF3 -> unconnected-(J1-Pin_37-Pad37)
- J1 pad 4: CLOCK -> unconnected-(J1-Pin_4-Pad4)
- J1 pad 5: ~CLEAR -> ~{CLEAR}
- J1 pad 6: ~DMA_IN -> unconnected-(J1-Pin_6-Pad6)
- J1 pad 8: ~DMA_OUT -> unconnected-(J1-Pin_8-Pad8)
- J1 pad 9: SC1 -> unconnected-(J1-Pin_9-Pad9)
- J2 pad 1: Net-(J2-Pad1) -> unconnected-(J2-Pad1)
- J2 pad 6: Net-(J2-Pad6) -> unconnected-(J2-Pad6)
- J2 pad 9: Net-(J2-Pad9) -> unconnected-(J2-Pad9)
- U3 pad 14: Net-(U3-Pad14) -> unconnected-(U3-FE-Pad14)
- U3 pad 15: Net-(U3-Pad15) -> unconnected-(U3-PE/OE-Pad15)
- U3 pad 21: ~CLEAR -> ~{CLEAR}
- U3 pad 22: Net-(U3-Pad22) -> unconnected-(U3-~{THRE}-Pad22)
- U3 pad 24: Net-(U3-Pad24) -> unconnected-(U3-~{RTS}-Pad24)
- U3 pad 36: Net-(U3-Pad36) -> unconnected-(U3-NC-Pad36)
- U4 pad 3: Net-(U4-Pad3) -> unconnected-(U4A-Q0-Pad3)
- U4 pad 6: Net-(U4-Pad6) -> unconnected-(U4A-Q3-Pad6)
- U5 pad 12: Net-(U5-Pad12) -> unconnected-(U5-Zd-Pad12)
- U5 pad 9: Net-(U5-Pad9) -> unconnected-(U5-Zc-Pad9)
- U6 pad 10: Net-(U6-Pad10) -> unconnected-(U6-SCL-Pad10)
- U6 pad 2: Net-(U6-Pad2) -> unconnected-(U6-GP0-Pad2)
- U6 pad 3: Net-(U6-Pad3) -> unconnected-(U6-GP1-Pad3)
- U6 pad 4: ~CLEAR -> Net-(U6-~{RST})
- U6 pad 7: Net-(U6-Pad7) -> unconnected-(U6-GP2-Pad7)
- U6 pad 8: Net-(U6-Pad8) -> unconnected-(U6-GP3-Pad8)
- U6 pad 9: Net-(U6-Pad9) -> unconnected-(U6-SDA-Pad9)
- X1 pad 1: Net-(X1-Pad1) -> unconnected-(X1-EN-Pad1)
Routing:
- net ~CLEAR: track 105.1 -> 0.00 mm
- net GND: track 340.5 -> 415.1 mm
- net ~{CLEAR}: track 0.00 -> 49.6 mm
- net VCC: track 171.3 -> 205.7 mm, vias 0 -> 1
- net High: track 161.8 -> 132.5 mm
- net /RTS: track 49.5 -> 70.0 mm
- net ~{N3}: track 47.2 -> 64.3 mm, vias 2 -> 0
- net /DTR: track 60.5 -> 44.9 mm
- net Q: track 51.3 -> 60.7 mm
- net Net-(U3-~{DA}): track 67.9 -> 76.2 mm
- net Net-(U3-~{CTS}): track 78.8 -> 70.7 mm
- net USB_D+: track 54.0 -> 47.2 mm, vias 0 -> 1
- net Net-(JP1-Pin_2): track 65.5 -> 71.3 mm
- net D6: track 38.8 -> 33.2 mm
- net Net-(JP1-Pin_6): track 28.0 -> 23.3 mm
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Other:
- net class Default removed
- net class Power removed
